File: kraft80/hardware/kraft80V2-ios.kicad_sch (KiCad schematic)
At the start: 49 parts, among them P1 100k, SW1 SW_Push, SW2 SW_Push, SW3 SW_Push, SW4 SW_Push, SW5 SW_Push, SW6 SW_Push, SW7 SW_Push, SW8 SW_Push, U10 74HC04, U11 74LS273, U3 74LS138, U4 4093, U5 74LS273, U6 74LS245, U7 74LS32, U93 74LS08, U97 74LS32, U99 74LS74

Commit message: Update Kraft80 Hardware Rev 2.2
Parts:
- removed U10: 74HC04, symbol 74xx:74HC04
- removed U4: 4093, symbol 4xxx:HEF4093B
- removed U7: 74LS32, symbol 74xx:74LS32
- removed U93: 74LS08, symbol 74xx:74LS08
- removed unit 5 of U97
- removed unit 3 of U99
- added JP1, JP2: Jumper_3_Bridged12, symbol Jumper:Jumper_3_Bridged12
- added JP10, JP11, JP12, JP13, JP8, JP9: SolderJumper_3_Open, symbol Jumper:SolderJumper_3_Open
- R10, R11, R12, R13, R14, R15, R21, R22, R8, R9: value 1k8 -> 2k
- R44: value 22 -> 22R
- renumbered C5 to C91, U3 to U91
Connections:
- net A4: now also JP11.1 (A); no longer U91.1 (A0)
- net A5: now also JP12.1 (A); no longer U91.2 (A1)
- net A6: now also JP13.1 (A); no longer U91.3 (A2)
- net GNDREF: now also JP1.2 (C), JP1.3 (B), JP2.2 (C), JP2.3 (B); no longer D10.1 (K), D3.1 (K), D4.1 (K), D5.1 (K), D6.1 (K), D7.1 (K), D8.1 (K), D9.1 (K)
- net ~{DISP_CS}: now also JP9.2 (C); no longer U91.14 (O1)
- net PA5: now reaches R9.1, U5.15 (Q5)
- net PA6: now reaches R10.1, U5.16 (Q6)
- net PB2: now reaches U11.6 (Q2)
- net PB3: now reaches U11.9 (Q3)
- net PA0: now reaches R12.1, U5.2 (Q0)
- net PA7: now reaches R11.1, U5.19 (Q7)
- net PA3: now reaches R15.1, U5.9 (Q3)
- net ~{CS2}: now reaches U91.13 (O2)
- net ~{CS2}: now also JP8.3 (B)
- net PA4: now reaches R8.1, U5.12 (Q4)
- net PA1: now reaches R13.1, U5.5 (Q1)
- net PA2: now reaches R14.1, U5.6 (Q2)
- net PC1: now reaches R22.1, U99.9 (Q)
- net CKKBD renamed CKPSHB
- net ~{FF_CS} renamed ~{CS4}
- net ~{CS4}: now also JP9.3 (B)
- removed net ~{LEDKB_CS}: U91.15 (O0), U97.12, U97.4
- new net: D3.1 (K), D4.1 (K), D5.1 (K), D6.1 (K), JP2.1 (A)
- new net: D10.1 (K), D7.1 (K), D8.1 (K), D9.1 (K), JP1.1 (A)
- new net: JP11.2 (C), U91.1 (A0)
- new net: JP12.2 (C), U91.2 (A1)
- new net: JP13.2 (C), U91.3 (A2)
- new net A0: JP11.3 (B)
- new net A1: JP12.3 (B)
- new net A2: JP13.3 (B)
- new net ~{CS0}: JP10.1 (A), JP8.1 (A), U91.15 (O0)
- new net ~{CS1}: JP10.3 (B), JP9.1 (A), U91.14 (O1)
- new net ~{LEDS_CS}: JP8.2 (C), U97.4
- new net ~{PSHB_CS}: JP10.2 (C), U97.12
Other:
- note added: "PORTS (KRAFT 80): 00h - LEDS(W) & BUTTONS(R) 10h - LCD(W) 40h - FFs(W) 50h - FPGA (VIDEO,SND,KBD)"
- note added: "PORTS (Z80 ALPHA): 01h - BUTTONS(R) 02h - LEDS(W) 04h - LCD(W)"
- note removed: "PORTS: 00h - LEDS(W) & BUTTONS(R) 10h - LCD(W) 20h - 8251(RW) 30h - 8259A(RW) 40h - FFs(W) 50h - FPGA (VIDEO,SND,KBD)"
- moved on the sheet: C17, C20, C9, C91, C97, P1, R44, RN1, SW1, SW2, SW3, SW4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
